File: CHAdeMO_V2.0.sch (KiCad schematic (older format))
At the start: 131 parts, among them IC1 ISO1050DUBR, IC2 ISO1050DUBR, J1 UJ2-BV-1-TH, J2 5810132011, J3 39-28-8020, J4 B2B-PH-K-S(LF)(SN), K1 V23086C1001A403-EV-BLBOX, Q1 IRLML0060TRPBF, Q2 IRLML0060TRPBF, Q3 IRLML0060TRPBF, Q4 IRLML0060TRPBF, Q5 DMP4065SQ-7, U1 M24M02-DRMN6TP, U2 ATSAM3X8EA-AU, U3 VOM617A-4T, U4 VOM617A-4T, U5 VOM617A-4T, U6 VOM617A-4T, U7 VOM617A-4T, Y1 CRYSTAL 12MHZ, Y2 Crystal 32.768kHz

Commit message: Dummy footprints
For stencil with cutouts for JLCPCB placed components
Parts:
- C1, C10, C11, C12, C14, C15, C16, C17, C18, C19, C20, C21, C22, C23, C24, C25, C26, C27, C28, C29, C30, C31, C32, C33, C36, C37, C42, C43, C45, C46, C47, C6, C7, C8, C9: footprint Capacitor_SMD:C_1206_3216Metric -> Components:DummyC1206_C_1206_3216Metric
- C13, C2, C3, C34, C35, C4, C5: footprint Capacitor_SMD:C_0603_1608Metric -> Components:Dummy_C_0603_1608Metric
- C38, C39, C40, C41: footprint Capacitor_SMD:C_0805_2012Metric -> Components:Dummy_C0805_210x135
- C44: footprint SamacSys_Parts:CAPAE1040X1050N -> Components:Dummy_ECAP_CAPAE1040X1050N
- D1, D2, D7, D8: footprint Diode_SMD:D_SOD-123 -> Components:Dummy_D_SOD-123
- L1, L2, L3, L4: footprint Inductor_SMD:L_0603_1608Metric -> Components:Dummy_L_0603_1608Metric
- L7, L8, L9: footprint Components:INDPM4442X200N -> Components:Dummy_L420_INDPM4442X200N
- LED1, LED2: footprint LED_SMD:LED_0603_1608Metric -> Components:Dummy_LED_0603_1608Metric
- R1, R14, R15, R16, R17, R18, R19, R2, R20, R21, R22, R23, R24, R25, R26, R27, R28, R29, R30, R4, R5, R8, R9: footprint Resistor_SMD:R_0805_2012Metric -> Components:Dummy_R_0805_2012Metric
- R3: footprint Resistor_SMD:R_0603_1608Metric -> Components:Dummy_R_0603_1608Metric
- R6, R7: footprint Resistor_SMD:R_1206_3216Metric -> Components:Dummy_R_1206_3216Metric
- U1: footprint SamacSys_Parts:SOIC127P600X175-8N -> Components:Dummy_SOIC8_SOIC127P600X175-8N
- Y1: footprint Crystal:Crystal_SMD_3225-4Pin_3.2x2.5mm -> Components:Dummy_Crystal_SMD_3225-4Pin_3.2x2.5mm
- Y2: footprint Crystal:Crystal_SMD_3215-2Pin_3.2x1.5mm -> Components:Dummy_Crystal_SMD_3215-2Pin_3.2x1.5mm
