File: CHAdeMO_V2.0.sch (KiCad schematic (older format))
At the start: 131 parts, among them IC1 ISO1050DUBR, IC2 ISO1050DUBR, J1 UJ2-BV-1-TH, J2 5810132011, J3 39-28-8020, J4 B2B-PH-K-S(LF)(SN), K1 V23086C1001A403-EV-BLBOX, Q1 IRLML0060TRPBF, Q2 IRLML0060TRPBF, Q3 IRLML0060TRPBF, Q4 IRLML0060TRPBF, Q5 DMP4065SQ-7, U1 M24M02-DRMN6TP, U2 ATSAM3X8EA-AU, U3 VOM617A-4T, U4 VOM617A-4T, U5 VOM617A-4T, U6 VOM617A-4T, U7 VOM617A-4T, Y1 CRYSTAL 12MHZ, Y2 Crystal 32.768kHz

Commit message: Prepare for 2.0.4
Parts:
- R17, R18: JLC-URL https://jlcpcb.com/parts/componentSearch?searchTxt=C38522 -> https://jlcpcb.com/parts/componentSearch?searchTxt=C25744; LCSC part number C38522 -> C25744; Stock type Extended -> Basic
- R19, R22, R23, R24, R27, R28, R9: JLC Footprint 0805 -> 0402; JLC-URL https://jlcpcb.com/parts/componentSearch?searchTxt=C38522 -> https://jlcpcb.com/parts/componentSearch?searchTxt=C25744; LCSC part number C38522 -> C25744; Stock type Extended -> Basic
- R21, R29: JLC-URL https://jlcpcb.com/parts/componentSearch?searchTxt=C27834 -> (none); LCSC part number C27834 -> (none)
- U2: LCSC part number (none) -> C79305

Commit message: Moved to LQFP100 chip
Parts:
- added IC3: ATSAM3X8CA-CU, SamacSys_Parts:BGA100C80P10X10_900X900X110, symbol SamacSys_Parts:ATSAM3X8CA-CU
Connections:
- net labels added: DFSDM, DFSDP, DHSDM, DHSDP, Xout
- wire segments 389 -> 410
Other:
- moved on the sheet: C11, C13, C18, C2, C3, C4, C5, L1, LED1, R1, R2, R3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

Commit message: V2.0.3 ordered at JLCPCB 23/12
Parts:
- removed C27: 100 nF, Capacitor_SMD:C_1206_3216Metric, symbol Device:C
- removed S1, S2: PTS647SM38SMTR2LFS, Components:PTS647SK38SMTR2LFS, symbol CHAdeMO_V2.0-rescue:PTS647SM38SMTR2LFS-PTS647SM38SMTR2LFS
- removed U2: ATSAM3X8EA-AU, Components:QFP50P2200X2200X145-144N, symbol CHAdeMO_V2.0-rescue:ATSAM3X8EA-AU-ATSAM3X8EA-AU
Connections:
- net labels removed: MASTER-RESET
- wire segments 410 -> 398
- no-connect marks 106 -> 61
Other:
- moved on the sheet: C11, C13, C18, C2, C28, C29, C3, C4, C5, IC3, L1, L4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
